Commit message: urdf: rotate force gripper connection -45deg

File: urdf/mycobot_320_pi_2022/mycobot_320_pi_2022_force_gripper.urdf (robot description, URDF)
Before this commit: robot firefighter, 15 links, 14 joints
Joints:
- joint joint6output_to_gripper_connect: origin xyz=0 0.0 0.0 rpy=0 0 0 -> xyz=0 0.0 0.0 rpy=0 0 -0.785398

Commit message: fix(urdf): scale collision meshes and add URDF tests
- Add scale=0.001 to collision meshes (mm -> m).

- Add ament pytest to validate URDF parsing, mesh paths, and absence of tcp_link.

File: urdf/mycobot_320_pi_2022/mycobot_320_pi_2022_force_gripper.urdf (robot description, URDF)
Before this commit: robot firefighter, 15 links, 14 joints
Links:
- link base: geometry collision mesh filename=package://mycobot320pi_urdf/urdf/mycobot_320_pi_2022/base.d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 scale=0.001 0.001 0.001; visual mesh filename=package://mycobot320pi_urdf/urdf/mycobot_320_pi_2022/base.d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
- link gripper_base: geometry collision mesh filename=package://mycobot320pi_urdf/urdf/mycobot_320_pi_2022/force_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 scale=0.001 0.001 0.001; visual mesh filename=package://mycobot320pi_urdf/urdf/mycobot_320_pi_2022/force_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
- link gripper_connection: geometry collision mesh filename=package://mycobot320pi_urdf/urdf/mycobot_320_pi_2022/force_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 scale=0.001 0.001 0.001; visual mesh filename=package://mycobot320pi_urdf/urdf/mycobot_320_pi_2022/force_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
- link gripper_left1: geometry collision mesh filename=package://mycobot320pi_urdf/urdf/mycobot_320_pi_2022/force_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 scale=0.001 0.001 0.001; visual mesh filename=package://mycobot320pi_urdf/urdf/mycobot_320_pi_2022/force_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
- link gripper_left2: geometry collision mesh filename=package://mycobot320pi_urdf/urdf/mycobot_320_pi_2022/force_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 scale=0.001 0.001 0.001; visual mesh filename=package://mycobot320pi_urdf/urdf/mycobot_320_pi_2022/force_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
- link gripper_left3: geometry collision mesh filename=package://mycobot320pi_urdf/urdf/mycobot_320_pi_2022/force_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 scale=0.001 0.001 0.001; visual mesh filename=package://mycobot320pi_urdf/urdf/mycobot_320_pi_2022/force_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
- link gripper_right1: geometry collision mesh filename=package://mycobot320pi_urdf/urdf/mycobot_320_pi_2022/force_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 scale=0.001 0.001 0.001; visual mesh filename=package://mycobot320pi_urdf/urdf/mycobot_320_pi_2022/force_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
- link gripper_right2: geometry collision mesh filename=package://mycobot320pi_urdf/urdf/mycobot_320_pi_2022/force_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 scale=0.001 0.001 0.001; visual mesh filename=package://mycobot320pi_urdf/urdf/mycobot_320_pi_2022/force_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
- link gripper_right3: geometry collision mesh filename=package://mycobot320pi_urdf/urdf/mycobot_320_pi_2022/force_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 scale=0.001 0.001 0.001; visual mesh filename=package://mycobot320pi_urdf/urdf/mycobot_320_pi_2022/force_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
- link link1: geometry collision mesh filename=package://mycobot320pi_urdf/urdf/mycobot_320_pi_2022/link1.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 scale=0.001 0.001 0.001; visual mesh filename=package://mycobot320pi_urdf/urdf/mycobot_320_pi_2022/link1.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
- link link2: geometry collision mesh filename=package://mycobot320pi_urdf/urdf/mycobot_320_pi_2022/link2.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 scale=0.001 0.001 0.001; visual mesh filename=package://mycobot320pi_urdf/urdf/mycobot_320_pi_2022/link2.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
- link link3: geometry collision mesh filename=package://mycobot320pi_urdf/urdf/mycobot_320_pi_2022/link3.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 scale=0.001 0.001 0.001; visual mesh filename=package://mycobot320pi_urdf/urdf/mycobot_320_pi_2022/link3.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
- link link4: geometry collision mesh filename=package://mycobot320pi_urdf/urdf/mycobot_320_pi_2022/link4.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 scale=0.001 0.001 0.001; visual mesh filename=package://mycobot320pi_urdf/urdf/mycobot_320_pi_2022/link4.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
- link link5: geometry collision mesh filename=package://mycobot320pi_urdf/urdf/mycobot_320_pi_2022/link5.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 scale=0.001 0.001 0.001; visual mesh filename=package://mycobot320pi_urdf/urdf/mycobot_320_pi_2022/link5.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
- link link6: geometry collision mesh filename=package://mycobot320pi_urdf/urdf/mycobot_320_pi_2022/link6.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 scale=0.001 0.001 0.001; visual mesh filename=package://mycobot320pi_urdf/urdf/mycobot_320_pi_2022/link6.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

Commit message: feat: add gripper_grasp frame

File: urdf/mycobot_320_pi_2022/mycobot_320_pi_2022_force_gripper.urdf (robot description, URDF)
Before this commit: robot firefighter, 15 links, 14 joints
Links:
- added link gripper_grasp
Joints:
- added joint gripper_base_to_gripper_grasp: type fixed, parent gripper_base, child gripper_grasp, origin xyz=0 0.1236 -0.02 rpy=-1.5708 0 0
